Commit message: dijkstra spp update

File: assets/2d_obs.urdf (robot description, URDF)
Before this commit: robot obs_box, 2 links, 1 joints
Links:
- link obs_box: geometry collision box size=0.05 0.05 0.05; visual box size=0.05 0.3 0.05

File: assets/roi_box.urdf (robot description, URDF)
Before this commit: robot roi_box, 2 links, 1 joints
Links:
- link roi_box: geometry visual box size=0.3 0.05 1.0
